File: docs/projects/can_servo/can_servo/can_servo.kicad_sch (KiCad schematic)
At the start: 19 parts, among them J1 Conn_01x02, J2 Conn_01x02, J3 Conn_01x03, U1 TPS54302, U10 TCAN330G, U11 C_100nF_0402, U12 C_4.7uF_0805, U13 C_100nF_0402, U14 C_100nF_0402, U15 C_100nF_0402, U16 R_10k_0402, U2 C_10uF_0805, U3 C_22uF_0805, U4 C_100nF_0402, U5 L_10uH_1210, U6 R_31.6k_0603, U7 R_10k_0603, U8 STM32G431CBUx, U9 AS5047D

Commit message: Regenerate examples + ELK layout tests
Re-execute power_brick / can_servo / sensor_node through the mandatory
ELK path; schematics now route with clean orthogonal wires that meet
pins, ERC clean (0 real / 0 expected on ERC_REAL_SYMBOL_CODES). Refresh
the tracked rendered SVGs.

Add tests/test_elk_layout.py: ELK raises LayoutError when node/the bridge
is unavailable (no fallback), and every routed wire is axis-aligned,
grid-snapped, and lands its pins on the routed endpoints.

Co-Authored-By: Claude Opus 4.8 (1M context) <noreply@anthropic.com>
Connections:
- net GND: now also J1.2 (Pin_2), J3.3 (Pin_3), U1.1 (GND), U10.2 (GND), U10.8 (S), U11.2, U12.2, U13.2, U14.2, U15.2, U2.2, U3.2, U7.2, U8.49 (VSS), U9.13 (GND), U9.5 (TST)
